Commit message: dodanie gazebo

File: src/mobil/urdf/mobile_robot.urdf.xacro (robot description, xacro)
@@ -7,6 +7,6 @@
     <color rgba="1 0 0 1"/>
   </material>
-  <material name="white">
-    <color rgba="1 1 1 1"/>
+  <material name="blue">
+    <color rgba="0 0 1 1"/>
   </material>
   <link name="obudowa">
@@ -25,5 +25,5 @@
     </collision>
     <inertial>
-      <mass value="1.0"/>
+      <mass value="10.0"/>
       <origin rpy="0 0 0" xyz="0 0 0"/>
       <inertia ixx="1" ixy="0" ixz="0" iyy="1" iyz="0" izz="1"/>
@@ -38,12 +38,12 @@
       <material name="red"/>
     </visual>
-    <visual>
+    <collision>
       <geometry>
         <cylinder radius="0.1" length="0.05"/>
       </geometry>
       <origin rpy="0 0 0" xyz="0 0 0"/>
-    </visual>
+    </collision>
     <inertial>
-      <mass value="1.0"/>
+      <mass value="2.5"/>
       <origin rpy="0 0 0" xyz="0 0 0"/>
       <inertia ixx="1" ixy="0" ixz="0" iyy="1" iyz="0" izz="1"/>
@@ -53,5 +53,5 @@
     <parent link="obudowa"/>
     <child link="kolo_lewe"/>
-    <origin xyz="0.125 0.125 0" rpy="-1.57 0 0"/>
+    <origin xyz="0.2 0.15 0" rpy="-1.57 0 0"/>
     <axis xyz="0 0 1"/>
   </joint>
@@ -64,12 +64,12 @@
       <material name="red"/>
     </visual>
-    <visual>
+    <collision>
       <geometry>
         <cylinder radius="0.1" length="0.05"/>
       </geometry>
       <origin rpy="0 0 0" xyz="0 0 0"/>
-    </visual>
+    </collision>
     <inertial>
-      <mass value="1.0"/>
+      <mass value="2.5"/>
       <origin rpy="0 0 0" xyz="0 0 0"/>
       <inertia ixx="1" ixy="0" ixz="0" iyy="1" iyz="0" izz="1"/>
@@ -79,19 +79,84 @@
     <parent link="obudowa"/>
     <child link="kolo_prawe"/>
-    <origin xyz="0.15 -0.125 0" rpy="-1.57 0 0"/>
+    <origin xyz="0.2 -0.15 0" rpy="-1.57 0 0"/>
     <axis xyz="0 0 1"/>
   </joint>
-  <link name="kula">
+  <link name="podpora">
     <visual>
-    <geometry>
-    <sphere radius="0.05"/>
-    </geometry>
-    <material name="white"/>
+      <geometry>
+        <sphere radius="0.1"/>
+      </geometry>
+      <origin rpy="0 0 0" xyz="0 0 0"/>
+      <material name="blue"/>
     </visual>
+    <collision>
+      <geometry>
+        <sphere radius="0.1"/>
+      </geometry>
+      <origin rpy="0 0 0" xyz="0 0 0"/>
+    </collision>
+    <inertial>
+      <mass value="1.0"/>
+      <origin rpy="0 0 0" xyz="0 0 0"/>
+      <inertia ixx="1" ixy="0" ixz="0" iyy="1" iyz="0" izz="1"/>
+    </inertial>
   </link>
-  <joint name="kula_buda" type="continuous">
+  <joint name="z_podpora" type="fixed">
     <parent link="obudowa"/>
-    <child link="kula"/>
-    <origin xyz="-0.17 0 -0.05"/>
+    <child link="podpora"/>
+    <origin xyz="-0.2 0 0" rpy="0 0 0"/>
+    <axis xyz="0 0 1"/>
   </joint>
+  <gazebo reference="kolo_lewe">
+    <mu1>0.1</mu1>
+    <mu2>0.1</mu2>
+    <kp>500000.0</kp>
+    <kd>10.0</kd>
+    <minDepth>0.001</minDepth>
+    <maxVel>0.1</maxVel>
+    <fdir1>1 0 0</fdir1>
+    <material>Gazebo/Green</material>
+  </gazebo>
+  <gazebo reference="kolo_prawe">
+    <mu1>0.1</mu1>
+    <mu2>0.1</mu2>
+    <kp>500000.0</kp>
+    <kd>10.0</kd>
+    <minDepth>0.001</minDepth>
+    <maxVel>0.1</maxVel>
+    <fdir1>1 0 0</fdir1>
+    <material>Gazebo/Red</material>
+  </gazebo>
+  <gazebo reference="podpora">
+    <mu1>0.01</mu1>
+    <mu2>0.01</mu2>
+    <kp>500000.0</kp>
+    <kd>10.0</kd>
+    <minDepth>0.001</minDepth>
+    <maxVel>0.1</maxVel>
+    <fdir1>1 0 0</fdir1>
+    <material>Gazebo/Blue</material>
+  </gazebo>
+  <gazebo>
+    <plugin name="moj_kontroler" filename="libgazebo_ros_diff_drive.so">
+      <commandTopic>cmd_vel</commandTopic>
+      <odometryTopic>odom</odometryTopic>
+      <odometryFrame>odom</odometryFrame>
+      <odometrySource>world</odometrySource>
+      <publishOdomTF>true</publishOdomTF>
+      <robotBaseFrame>obudowa</robotBaseFrame>
+      <publishWheelTF>false</publishWheelTF>
+      <publishTf>true</publishTf>
+      <publishWheelJointState>true</publishWheelJointState>
+      <legacyMode>false</legacyMode>
+      <updateRate>30</updateRate>
+      <leftJoint>z_kolo_lewe</leftJoint>
+      <rightJoint>z_kolo_prawe</rightJoint>
+      <wheelSeparation>0.3</wheelSeparation>
+      <wheelDiameter>0.2</wheelDiameter>
+      <wheelAcceleration>1</wheelAcceleration>
+      <wheelTorque>10</wheelTorque>
+      <rosDebugLevel>na</rosDebugLevel>
+    </plugin>
+  </gazebo>
 </robot>

Commit message: kamera lidar imu

File: src/mobil/urdf/mobile_robot.urdf.xacro (robot description, xacro)
@@ -10,4 +10,7 @@
     <color rgba="0 0 1 1"/>
   </material>
+  <material name="black">
+    <color rgba="1 1 1 1"/>
+  </material>
   <link name="obudowa">
     <visual>
@@ -27,5 +30,5 @@
       <mass value="10.0"/>
       <origin rpy="0 0 0" xyz="0 0 0"/>
-      <inertia ixx="1" ixy="0" ixz="0" iyy="1" iyz="0" izz="1"/>
+      <inertia ixx="2E-07" ixy="0" ixz="0" iyy="1E-06" iyz="0" izz="1E-06"/>
     </inertial>
   </link>
@@ -47,5 +50,5 @@
       <mass value="2.5"/>
       <origin rpy="0 0 0" xyz="0 0 0"/>
-      <inertia ixx="1" ixy="0" ixz="0" iyy="1" iyz="0" izz="1"/>
+      <inertia ixx="1E-03" ixy="0" ixz="0" iyy="1E-03" iyz="0" izz="1E-03"/>
     </inertial>
   </link>
@@ -73,5 +76,5 @@
       <mass value="2.5"/>
       <origin rpy="0 0 0" xyz="0 0 0"/>
-      <inertia ixx="1" ixy="0" ixz="0" iyy="1" iyz="0" izz="1"/>
+      <inertia ixx="1E-03" ixy="0" ixz="0" iyy="1E-03" iyz="0" izz="1E-03"/>
     </inertial>
   </link>
@@ -99,5 +102,5 @@
       <mass value="1.0"/>
       <origin rpy="0 0 0" xyz="0 0 0"/>
-      <inertia ixx="1" ixy="0" ixz="0" iyy="1" iyz="0" izz="1"/>
+      <inertia ixx="1E-03" ixy="0" ixz="0" iyy="1E-03" iyz="0" izz="1E-03"/>
     </inertial>
   </link>
@@ -107,4 +110,61 @@
     <origin xyz="-0.2 0 0" rpy="0 0 0"/>
     <axis xyz="0 0 1"/>
+  </joint>
+  <link name="imu_link"/>
+  <joint name="imu_joint" type="fixed">
+    <parent link="obudowa"/>
+    <child link="imu_link"/>
+    <origin xyz="0.2 0.0 0.0" rpy="0.0 0.0 0.0"/>
+    <axis xyz="0.0 0.0 1.0"/>
+  </joint>
+  <link name="lidar">
+    <visual>
+      <origin xyz="0.2 0 -0.05" rpy="0 0 0"/>
+      <geometry>
+        <cylinder radius="0.025" length="0.1"/>
+      </geometry>
+      <material name="black"/>
+    </visual>
+    <collision>
+      <origin xyz="0.2 0 -0.05" rpy="0 0 0"/>
+      <geometry>
+        <cylinder radius="0.025" length="0.1"/>
+      </geometry>
+    </collision>
+    <inertial>
+      <origin xyz="0.2 0 -0.05" rpy="0 0 0"/>
+      <mass value="0.1"/>
+      <inertia ixx="0.001" ixy="0" ixz="0" iyy="0.001" iyz="0" izz="0.001"/>
+    </inertial>
+  </link>
+  <joint name="lidar_joint" type="fixed">
+    <parent link="obudowa"/>
+    <child link="lidar"/>
+    <origin xyz="0 0 0.15" rpy="0 0 0"/>
+  </joint>
+  <link name="kamera">
+    <visual>
+      <origin xyz="-0.0125 0 0" rpy="0 0 0"/>
+      <geometry>
+        <box size="0.025 0.05 0.05"/>
+      </geometry>
+      <material name="black"/>
+    </visual>
+    <collision>
+      <origin xyz="-0.0125 0 0" rpy="0 0 0"/>
+      <geometry>
+        <box size="0.025 0.05 0.05"/>
+      </geometry>
+    </collision>
+    <inertial>
+      <origin xyz="0 0 -0.05" rpy="0 0 0"/>
+      <mass value="0.1"/>
+      <inertia ixx="0.001" ixy="0" ixz="0" iyy="0.001" iyz="0" izz="0.001"/>
+    </inertial>
+  </link>
+  <joint name="kamera_joint" type="fixed">
+    <parent link="obudowa"/>
+    <child link="kamera"/>
+    <origin xyz="0.275 0 0" rpy="0 0 0"/>
   </joint>
   <gazebo reference="kolo_lewe">
@@ -137,4 +197,80 @@
     <fdir1>1 0 0</fdir1>
     <material>Gazebo/Blue</material>
+  </gazebo>
+  <gazebo reference="imu_link">
+    <sensor type="imu" name="imu">
+      <always_on>true</always_on>
+      <visualize>true</visualize>
+    </sensor>
+    <material>Gazebo/FlatBlack</material>
+  </gazebo>
+  <gazebo reference="lidar">
+    <material>Gazebo/FlatBlack</material>
+    <sensor type="ray" name="lds_lfcd_sensor">
+      <pose>0 0 0 0 0 0</pose>
+      <visualize>true</visualize>
+      <update_rate>5</update_rate>
+      <ray>
+        <scan>
+          <horizontal>
+            <samples>360</samples>
+            <resolution>1</resolution>
+            <min_angle>0.0</min_angle>
+            <max_angle>6.28319</max_angle>
+          </horizontal>
+        </scan>
+        <range>
+          <min>0.120</min>
+          <max>16</max>
+          <resolution>0.01</resolution>
+        </range>
+        <noise>
+          <type>gaussian</type>
+          <mean>0.0</mean>
+          <stddev>0.02</stddev>
+        </noise>
+      </ray>
+      <plugin name="gazebo_ros_lds_lfcd_controller" filename="libgazebo_ros_laser.so">
+        <topicName>laser_scan</topicName>
+        <frameName>lidar</frameName>
+      </plugin>
+    </sensor>
+</gazebo>
+<gazebo reference="kamera">
+    <sensor type="camera" name="camera1">
+      <update_rate>30.0</update_rate>
+      <camera name="head">
+        <horizontal_fov>1.3962634</horizontal_fov>
+        <image>
+          <width>640</width>
+          <height>480</height>
+          <format>R8G8B8</format>
+        </image>
+        <clip>
+          <near>0.02</near>
+          <far>300</far>
+        </clip>
+        <noise>
+          <type>gaussian</type>
+          <mean>0.0</mean>
+          <stddev>0.007</stddev>
+        </noise>
+      </camera>
+      <plugin name="camera_controller" filename="libgazebo_ros_camera.so">
+        <alwaysOn>true</alwaysOn>
+        <updateRate>0.0</updateRate>
+        <cameraName>camera1</cameraName>
+        <imageTopicName>image_raw</imageTopicName>
+        <cameraInfoTopicName>camera_info</cameraInfoTopicName>
+        <frameName>kamera</frameName>
+        <hackBaseline>0.07</hackBaseline>
+        <distortionK1>0.0</distortionK1>
+        <distortionK2>0.0</distortionK2>
+        <distortionK3>0.0</distortionK3>
+        <distortionT1>0.0</distortionT1>
+        <distortionT2>0.0</distortionT2>
+      </plugin>
+      <visualize>true</visualize>
+    </sensor>
   </gazebo>
   <gazebo>
@@ -159,4 +295,30 @@
       <rosDebugLevel>na</rosDebugLevel>
     </plugin>
+    <plugin name="imu_plugin" filename="libgazebo_ros_imu.so">
+      <alwaysOn>true</alwaysOn>
+      <bodyName>imu_link</bodyName>
+      <frameName>imu_link</frameName>
+      <topicName>imu</topicName>
+      <serviceName>imu_service</serviceName>
+      <gaussianNoise>0.0</gaussianNoise>
+      <updateRate>200</updateRate>
+      <imu>
+        <noise>
+          <type>gaussian</type>
+          <rate>
+            <mean>0.0</mean>
+            <stddev>2e-4</stddev>
+            <bias_mean>0.0000075</bias_mean>
+            <bias_stddev>0.0000008</bias_stddev>
+          </rate>
+          <accel>
+            <mean>0.0</mean>
+            <stddev>1.7e-2</stddev>
+            <bias_mean>0.1</bias_mean>
+            <bias_stddev>0.001</bias_stddev>
+          </accel>
+        </noise>
+      </imu>
+    </plugin>
   </gazebo>
 </robot>

Commit message: skonczenie projektu nr2

File: src/mobil/urdf/mobile_robot.urdf.xacro (robot description, xacro)
@@ -50,5 +50,5 @@
       <mass value="2.5"/>
       <origin rpy="0 0 0" xyz="0 0 0"/>
-      <inertia ixx="1E-03" ixy="0" ixz="0" iyy="1E-03" iyz="0" izz="1E-03"/>
+      <inertia ixx="1E-05" ixy="0" ixz="0" iyy="1E-05" iyz="0" izz="1E-05"/>
     </inertial>
   </link>
@@ -76,5 +76,5 @@
       <mass value="2.5"/>
       <origin rpy="0 0 0" xyz="0 0 0"/>
-      <inertia ixx="1E-03" ixy="0" ixz="0" iyy="1E-03" iyz="0" izz="1E-03"/>
+      <inertia ixx="1E-05" ixy="0" ixz="0" iyy="1E-05" iyz="0" izz="1E-05"/>
     </inertial>
   </link>
@@ -102,5 +102,5 @@
       <mass value="1.0"/>
       <origin rpy="0 0 0" xyz="0 0 0"/>
-      <inertia ixx="1E-03" ixy="0" ixz="0" iyy="1E-03" iyz="0" izz="1E-03"/>
+      <inertia ixx="1E-05" ixy="0" ixz="0" iyy="1E-05" iyz="0" izz="1E-05"/>
     </inertial>
   </link>
